Commit message: miss change and I am just change it back to the former files

File: urdf/robot.xacro (robot description, xacro)
@@ -3,20 +3,4 @@
   <!-- Mass parameters -->
   <xacro:property name="pi" value="3.14159265" />
-  <!-- Include the XACRO file that defines a Hokuyo LIDAR. -->
-  <xacro:include filename="$(find
-  gazebo_plugins)/test/multi_robot_scenario/xacro/laser/hokuyo.xacro" />
-  <xacro:laser name="laser_vert_bottom" parent="base" xyz="0.3157894464801903
-  -0.002068548615034871 0.5099999434059285" rpy="3.1354753 -1.3045001 0.0024658"
-  meshes="package://gazebo_plugins/test/multi_robot_scenario/meshes/laser" />
-  <xacro:laser name="laser_vert_top_right" parent="base"  xyz="0.2978 -0.1450 1.8451" rpy="-1.1760 0.6313 -1.9377" meshes="package://gazebo_plugins/test/multi_robot_scenario/meshes/laser" />
-  <xacro:laser name="laser_vert_top_left" parent="base"  xyz="0.2997 0.1531 1.8443" rpy="1.1780 0.6198 1.9560" meshes="package://gazebo_plugins/test/multi_robot_scenario/meshes/laser" />
-  <!-- Include the XACRO file that defines a Hokuyo LIDAR. -->
-  <xacro:include filename="$(find velodyne_description)/urdf/VLP-16.urdf.xacro"/>
-  <!-- Invoke the macro to define the Hokuyo LIDAR. -->
-  <xacro:VLP-16 parent="base" name="laser_horiz" topic="laser_horiz/packets" hz="10"
-samples="440" gpu="false">
-  <origin xyz="0.2325416305773505 -0.0001380069427607134 1.920122926231907"
-rpy="-0.0012068 0.114646 -0.0015308" />
-  </xacro:VLP-16>
   <!-- XACRO Macro definition block to add around the wheel link and joint !-->
   <xacro:macro name="xacro_name" params="side reflect">
@@ -58,52 +42,4 @@
     </collision>
   </link>
-  <link name="laser_vert_bottom_joint">
-    <visual>
-      <geometry>
-        <box size="0.062 0.062 0.087" />
-      </geometry>
-    </visual>
-    <collision>
-      <geometry>
-        <box size="0.062 0.062 0.087" />
-      </geometry>
-    </collision>
-  </link>
-  <link name="laser_vert_top_right_joint">
-    <visual>
-      <geometry>
-        <box size="0.062 0.062 0.087" />
-      </geometry>
-    </visual>
-    <collision>
-      <geometry>
-        <box size="0.062 0.062 0.087" />
-      </geometry>
-    </collision>
-  </link>
-  <link name="laser_vert_top_left_joint">
-    <visual>
-      <geometry>
-        <box size="0.062 0.062 0.087" />
-      </geometry>
-    </visual>
-    <collision>
-      <geometry>
-        <box size="0.062 0.062 0.087" />
-      </geometry>
-    </collision>
-  </link>
-  <link name="laser_horiz_joint">
-    <visual>
-      <geometry>
-        <cylinder radius="0.052" length="0.072" />
-      </geometry>
-    </visual>
-    <collision>
-      <geometry>
-        <cylinder radius="0.052" length="0.072" />
-      </geometry>
-    </collision>
-  </link>
   <link name="wheel_center_joint">
     <visual>
@@ -118,24 +54,4 @@
     </collision>
   </link>
-  <joint name="base_laser_vert_bottom_joint" type="fixed">
-    <parent link="base" />
-    <child link="laser_vert_bottom_joint" />
-      <origin xyz="0.3158 -0.0021 0.5100" rpy="3.1355 -1.3045 0.0025" />
-  </joint>
-  <joint name="base_laser_vert_top_right_joint" type="fixed">
-    <parent link="base" />
-    <child link="laser_vert_top_right_joint" />
-    <origin xyz="0.2978 -0.1450 1.8451" rpy="-1.1760 0.6313 -1.9377" />
-</joint>
-  <joint name="base_laser_vert_top_left_joint" type="fixed">
-    <parent link="base" />
-    <child link="laser_vert_top_left_joint" />
-      <origin xyz="0.2997 0.1531 1.8443" rpy="1.1780 0.6198 1.9560" />
-  </joint>
-  <joint name="base_laser_horiz_joint" type="fixed">
-    <parent link="base" />
-    <child link="laser_horiz_joint" />
-      <origin xyz="0.2325 0.0001 1.9201" rpy="-0.0012 0.1146 -0.0015" />
-  </joint>
   <joint name="base_wheel_center_joint" type="fixed">
     <parent link="base" />
@@ -143,3 +59,19 @@
     <origin xyz="0.10 0.0 -0.05" rpy="${-pi/2} 0.0 0.0" />
   </joint>
+<!-- Include the XACRO file that defines a Hokuyo LIDAR. -->
+  <xacro:include filename="$(find
+  gazebo_plugins)/test/multi_robot_scenario/xacro/laser/hokuyo.xacro" />
+  <xacro:laser name="laser_vert_bottom" parent="base" xyz="0.3157894464801903
+  -0.002068548615034871 0.5099999434059285" rpy="3.1354753 -1.3045001 0.0024658"
+  meshes="package://gazebo_plugins/test/multi_robot_scenario/meshes/laser" />
+  <xacro:laser name="laser_vert_top_right" parent="base"  xyz="0.2978 -0.1450 1.8451" rpy="-1.1760 0.6313 -1.9377" meshes="package://gazebo_plugins/test/multi_robot_scenario/meshes/laser" />
+  <xacro:laser name="laser_vert_top_left" parent="base"  xyz="0.2997 0.1531 1.8443" rpy="1.1780 0.6198 1.9560" meshes="package://gazebo_plugins/test/multi_robot_scenario/meshes/laser" />
+  <!-- Include the XACRO file that defines a Hokuyo LIDAR. -->
+  <xacro:include filename="$(find velodyne_description)/urdf/VLP-16.urdf.xacro"/>
+  <!-- Invoke the macro to define the Hokuyo LIDAR. -->
+  <xacro:VLP-16 parent="base" name="laser_horiz" topic="laser_horiz/packets" hz="10"
+samples="440" gpu="false">
+  <origin xyz="0.2325416305773505 -0.0001380069427607134 1.920122926231907"
+rpy="-0.0012068 0.114646 -0.0015308" />
+  </xacro:VLP-16>
 </robot>
